Commit message: updated peg vel and env setup

File: pybulletgym/envs/assets/urdf/cuboid_peg.urdf (robot description, URDF)
Before this commit: robot cuboid_peg, 5 links, 4 joints
Joints:
- joint x_slider: limit lower=-0.5 upper=0.5 effort=10000 velocity=1. -> lower=-0.5 upper=0.5 effort=10000 velocity=2.
- joint y_slider: limit lower=-0.5 upper=0.5 effort=10000 velocity=1. -> lower=-0.5 upper=0.5 effort=10000 velocity=2.
- joint z_axis_joint: limit lower=-3.14 upper=3.14 effort=10000 velocity=1. -> lower=-3.14 upper=3.14 effort=10000 velocity=3.

File: pybulletgym/envs/assets/urdf/hole.urdf (robot description, URDF)
Before this commit: robot hole, 5 links, 4 joints
Links:
- added link hole_left, mass 1.0; collision box size=0.44 0.1 0.053; visual box size=0.44 0.1 0.053
- added link hole_right, mass 1.0; collision box size=0.44 0.1 0.053; visual box size=0.44 0.1 0.053
Joints:
- added joint hole_left_joint: type fixed, parent world, child hole_left
- added joint hole_right_joint: type fixed, parent world, child hole_right
