Commit message: lowered the max vel for shallow hole

File: pybulletgym/envs/assets/urdf/cuboid_thin_peg.urdf (robot description, URDF)
Before this commit: robot cuboid_peg, 5 links, 4 joints
Joints:
- joint x_slider: limit lower=-0.475 upper=0.475 effort=10000 velocity=2. -> lower=-0.475 upper=0.475 effort=10000 velocity=0.1
- joint y_slider: limit lower=-0.475 upper=0.475 effort=10000 velocity=2. -> lower=-0.475 upper=0.475 effort=10000 velocity=0.1
- joint z_axis_joint: limit lower=-3.14 upper=3.14 effort=10000 velocity=3. -> lower=-3.14 upper=3.14 effort=10000 velocity=1.

File: pybulletgym/envs/assets/urdf/shallow_hole.urdf (robot description, URDF)
Before this commit: robot hole, 7 links, 6 joints
Links:
- link wall_left: geometry collision box size=0.5 0.02 0.05; visual box size=0.5 0.02 0.05
- link wall_right: geometry collision box size=0.5 0.02 0.05; visual box size=0.5 0.02 0.05
- link wall_up: geometry collision box size=0.5 0.02 0.05; visual box size=0.5 0.02 0.05
