Commit message: added peginhole with a gripper

File: pybulletgym/envs/assets/robots/peg/peg_description/peg_in_shallow_hole.urdf (robot description, URDF)
Before this commit: robot hole, 7 links, 6 joints
Links:
- added link peg, mass 1.0; collision box size=0.1 0.02 0.05; visual box size=0.1 0.02 0.05
- added link target, mass 0.00001; visual box size=0.1 0.02 0.05
Joints:
- added joint peg_joint: type planar, parent world, child peg, origin xyz=0 0 0 rpy=0.0 0.0 0.0, axis 0 0 1, limit effort=100000000000 velocity=1000000000
- added joint target_joint: type fixed, parent world, child target, origin xyz=0 -0.2375 0 rpy=0.0 0.0 0.0
