Commit message: first success version with multimodal observations

File: pybulletgym/envs/assets/robots/peg/peg_description/capsule_thin_peg.urdf (robot description, URDF)
Before this commit: robot cuboid_peg, 6 links, 5 joints
Links:
- link peg: mass 0.1 -> 1.01
- link peg_right: geometry collision cylinder length=0.05 radius=0.01; visual cylinder length=0.05 radius=0.01
Joints:
- joint peg_left_joint: origin xyz=0 0 0 rpy=0.0 0.0 0.0 -> xyz=-0.04 0 0 rpy=0.0 0.0 0.0
- joint peg_right_joint: origin xyz=0 0 0 rpy=0.0 0.0 0.0 -> xyz=0.04 0 0 rpy=0 0 0

File: pybulletgym/envs/assets/robots/peg/peg_description/shallow_hole.urdf (robot description, URDF)
Before this commit: robot hole, 8 links, 7 joints
Links:
- link target: geometry 
- link wall_left: geometry collision box size=0.5 0.02 0.05
- link wall_right: geometry collision box size=0.5 0.02 0.05
- link wall_up: geometry collision box size=0.5 0.02 0.05
Joints:
- joint target_joint: origin xyz=0 -0.2375 0 rpy=0.0 0.0 0.0 -> xyz=0 -0.24 0 rpy=0.0 0.0 0.0
