Commit message: short gripper

File: pybulletgym/envs/assets/robots/gripper/gripper_description/simple_gripper.urdf (robot description, URDF)
Before this commit: robot gripper, 8 links, 7 joints
Links:
- link left_finger: geometry collision box size=0.01 0.01 0.05; visual box size=0.01 0.01 0.05
- link right_finger: geometry collision box size=0.01 0.01 0.05; visual box size=0.01 0.01 0.05

Commit message: adjusted finger length

File: pybulletgym/envs/assets/robots/gripper/gripper_description/simple_gripper.urdf (robot description, URDF)
Before this commit: robot gripper, 8 links, 7 joints
Links:
- link left_finger: geometry collision box size=0.02 0.01 0.05; visual box size=0.02 0.01 0.05
- link right_finger: geometry collision box size=0.02 0.01 0.05; visual box size=0.02 0.01 0.05

Commit message: capsule peg

File: pybulletgym/envs/assets/robots/gripper/gripper_description/simple_gripper.urdf (robot description, URDF)
Before this commit: robot gripper, 8 links, 7 joints
Links:
- link left_finger: geometry collision box size=0.02 0.005 0.05; visual box size=0.02 0.005 0.05
- link left_knuckle: mass 0.5 -> 0.001; geometry 
- link palm: geometry collision box size=0.005 0.04 0.05; visual box size=0.005 0.04 0.05
- link right_finger: geometry collision box size=0.02 0.005 0.05; visual box size=0.02 0.005 0.05
- link right_knuckle: mass 0.5 -> 0.001; geometry 
Joints:
- joint left_finger_joint: axis 0 1 0 -> 0 -1 0; limit lower=0.005 upper=0.03 effort=0 velocity=0 -> lower=0.0 upper=0.04 effort=2 velocity=0; origin xyz=0 0 0 rpy=0.0 0.0 0.0 -> xyz=0 0 0 rpy=0 0 0
- joint left_link_joint: origin xyz=0 0.005 0 rpy=0.0 0.0 0.0 -> xyz=0 0 0 rpy=0 0 0
- joint right_finger_joint: axis 0 -1 0 -> 0 1 0; limit lower=0.005 upper=0.03 effort=0 velocity=0 -> lower=0.0 upper=0.04 effort=1000 velocity=0; origin xyz=0 0 0 rpy=0.0 0.0 0.0 -> xyz=0 0 0 rpy=0 0 0
- joint right_link_joint: origin xyz=0 -0.005 0 rpy=0.0 0.0 0.0 -> xyz=0 0 0 rpy=0.0 0.0 0.0
- joint x_slider: limit lower=-0.25 upper=0.25 effort=1000 velocity=0.01 -> lower=-0.25 upper=0.25 effort=1000 velocity=0.001
- joint y_slider: limit lower=-0.25 upper=0.25 effort=1000 velocity=0.01 -> lower=-0.25 upper=0.25 effort=1000 velocity=0.001
- joint z_axis_joint: limit lower=-3.14 upper=3.14 effort=1000 velocity=0.5 -> lower=-3.14 upper=3.14 effort=1000 velocity=0.05

File: pybulletgym/envs/assets/robots/peg/peg_description/capsule_thin_peg.urdf (robot description, URDF)
Before this commit: robot cuboid_peg, 4 links, 3 joints
Links:
- added link peg_left, mass 0.000001; collision cylinder length=0.05 radius=0.01; visual cylinder length=0.05 radius=0.01
- added link peg_right, mass 0.000001; collision cylinder length=0.05 radius=0.000091; visual cylinder length=0.05 radius=0.0091
- link peg: geometry collision box size=0.08 0.02 0.05; visual box size=0.08 0.02 0.05
Joints:
- added joint peg_left_joint: type fixed, parent peg, child peg_left, origin xyz=0 0 0 rpy=0.0 0.0 0.0
- added joint peg_right_joint: type fixed, parent peg, child peg_right, origin xyz=0 0 0 rpy=0.0 0.0 0.0

Commit message: adjusted gripper

File: pybulletgym/envs/assets/robots/gripper/gripper_description/simple_gripper.urdf (robot description, URDF)
Before this commit: robot gripper, 8 links, 7 joints
Links:
- link left_finger: geometry collision box size=0.03 0.005 0.05; visual box size=0.03 0.005 0.05
- link palm: geometry collision box size=0.025 0.04 0.05; visual box size=0.025 0.04 0.05
- link right_finger: geometry collision box size=0.03 0.005 0.05; visual box size=0.03 0.005 0.05
Joints:
- joint left_finger_joint: limit lower=0.0 upper=0.04 effort=2 velocity=0 -> lower=0.01 upper=0.04 effort=2 velocity=0
- joint x_slider: limit lower=-0.25 upper=0.25 effort=1000 velocity=0.001 -> lower=-0.25 upper=0.25 effort=1000 velocity=0.005
- joint y_slider: limit lower=-0.25 upper=0.25 effort=1000 velocity=0.001 -> lower=-0.25 upper=0.25 effort=1000 velocity=0.005
- joint z_axis_joint: limit lower=-3.14 upper=3.14 effort=1000 velocity=0.05 -> lower=-3.14 upper=3.14 effort=1000 velocity=0.08

Commit message: release reward

File: pybulletgym/envs/assets/robots/gripper/gripper_description/simple_gripper.urdf (robot description, URDF)
Before this commit: robot gripper, 8 links, 7 joints
Joints:
- joint left_finger_joint: limit lower=0.01 upper=0.04 effort=2 velocity=0 -> lower=0.01 upper=0.04 effort=2 velocity=0.005
- joint right_finger_joint: limit lower=0.0 upper=0.04 effort=1000 velocity=0 -> lower=0.0 upper=0.04 effort=1000 velocity=0.005
